File: testsmt/testsmt.kicad_pcb (KiCad board)
At the start: 2 copper layers, 47 parts, among them J1 DIN-5_180degree, J2 Conn_01x16, J3 Conn_01x16, J4 Conn_01x16, J5 AudioJack3_Ground_Switch, U1 6N138, U2 Teensy3.2, U3 4051, U4 4051, U5 4051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

Commit message: about to try out some routing
Parts:
- moved R4 169.9 mm to (190.3, 86.1)
- moved R6 169.9 mm to (193.9, 86.1)
- moved R7 136.9 mm to (200.9, 90.0)
- moved U7 107.8 mm to (157.5, 66.5)
- moved RV1 104.0 mm to (52.9, 111.9), turned to 90 degrees
- moved RV3 104.0 mm to (96.1, 111.9), turned to 90 degrees
- moved RV4 104.0 mm to (116.4, 111.9), turned to 90 degrees
- moved RV5 104.0 mm to (136.8, 111.9), turned to 90 degrees
- moved RV2 104.0 mm to (73.3, 111.9), turned to 90 degrees
- moved RV6 104.0 mm to (157.1, 111.9), turned to 90 degrees
- moved R5 103.9 mm to (180.0, 90.0)
- moved C2 98.6 mm to (149.0, 33.4), turned to 90 degrees
- moved RV7 73.7 mm to (159.0, 53.0)
- moved J1 73.1 mm to (126.0, 35.0)
- moved D2 72.4 mm to (117.0, 58.4)
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Routing:
- added copper zone on B.Cu, net GND
- added copper zone on F.Cu, net GND
Other:
- board outline added: 200 x 100 mm

Commit message: started routing
Parts:
- moved U6 27.6 mm to (93.0, 91.0)
- moved U4 17.6 mm to (93.0, 76.0)
Routing:
- net /CHANNEL_0: track 0.00 -> 51.0 mm
- net /CHANNEL_1: track 0.00 -> 48.9 mm, vias 0 -> 1
- net +3V3: track 0.00 -> 38.8 mm
- net /SHIFT_REG_LATCH: track 0.00 -> 35.4 mm
- net Net-(R8-Pad2): track 0.00 -> 30.4 mm, vias 0 -> 2
- net Net-(R9-Pad2): track 0.00 -> 26.1 mm
- net /SHIFT_REG_CLOCK: track 0.00 -> 25.7 mm
- net /SHIFT_REG_DATA: track 0.00 -> 24.1 mm
- net Net-(R10-Pad2): track 0.00 -> 22.2 mm
- net Net-(R11-Pad2): track 0.00 -> 18.1 mm
- net Net-(R12-Pad2): track 0.00 -> 14.8 mm
- net Net-(R15-Pad2): track 0.00 -> 13.8 mm, vias 0 -> 2
- net Net-(R13-Pad2): track 0.00 -> 12.9 mm, vias 0 -> 2
- net Net-(R14-Pad2): track 0.00 -> 11.3 mm, vias 0 -> 2
- net /CHANNEL_9: track 0.00 -> 7.20 mm
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
Commit message: routing going well
Routing:
- net /ADDRESS_READ_C: track 0.00 -> 64.7 mm, vias 0 -> 1
- net /ADDRESS_READ_B: track 0.00 -> 58.7 mm, vias 0 -> 3
- net /ADDRESS_READ_A: track 0.00 -> 56.5 mm
- net /CHANNEL_12: track 7.20 -> 57.4 mm
- net /CHANNEL_4: track 7.20 -> 52.1 mm
- net /CHANNEL_6: track 7.20 -> 50.5 mm
- net /CHANNEL_9: track 7.20 -> 50.3 mm
- net /CHANNEL_2: track 7.20 -> 49.1 mm, vias 0 -> 1
- net /CHANNEL_8: track 7.20 -> 47.5 mm
- net /CHANNEL_3: track 7.20 -> 47.0 mm
- net /CHANNEL_11: track 7.20 -> 44.5 mm
- net /CHANNEL_10: track 7.20 -> 44.3 mm, vias 0 -> 1
- net /CHANNEL_7: track 7.20 -> 41.0 mm
- net /CHANNEL_5: track 7.20 -> 39.2 mm
- net /CONNECTION_READ_A: track 0.00 -> 31.9 mm, vias 0 -> 1
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
Commit message: routing...
Parts:
- moved U3 99.2 mm to (54.0, 48.0)
- moved U5 79.4 mm to (54.0, 77.0)
- moved U4 57.3 mm to (54.0, 34.0)
- moved D3 56.7 mm to (87.9, -4.30)
- moved R8 56.7 mm to (87.9, 0.78)
- moved D10 56.7 mm to (123.5, -4.30)
- moved D4 56.7 mm to (93.0, -4.30)
- moved D5 56.7 mm to (98.1, -4.30)
- moved D6 56.7 mm to (103.2, -4.30)
- moved D7 56.7 mm to (108.2, -4.30)
- moved D8 56.7 mm to (113.3, -4.30)
- moved D9 56.7 mm to (118.4, -4.30)
- moved R10 56.7 mm to (98.1, 0.78)
- moved R11 56.7 mm to (103.2, 0.78)
- moved R12 56.7 mm to (108.2, 0.78)
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Routing:
- net /ADDRESS_SEND_A: track 0.00 -> 67.8 mm
- net /ADDRESS_SEND_B: track 0.00 -> 59.4 mm
- net /CHANNEL_12: track 57.4 -> 3.60 mm
- net /ADDRESS_SEND_C: track 0.00 -> 50.8 mm
- net /CONNECTION_READ_A: track 31.9 -> 80.1 mm, vias 1 -> 0
- net /CHANNEL_9: track 50.3 -> 3.60 mm
- net /CHANNEL_8: track 47.5 -> 3.60 mm
- net /CHANNEL_11: track 44.5 -> 3.60 mm
- net /CHANNEL_10: track 44.3 -> 3.60 mm, vias 1 -> 0
- net +3V3: track 38.8 -> 0.00 mm
- net /CHANNEL_7: track 41.0 -> 3.60 mm
- net /SHIFT_REG_LATCH: track 35.4 -> 0.00 mm
- net /CHANNEL_15: track 38.8 -> 3.60 mm
- net /CHANNEL_13: track 37.0 -> 3.60 mm
- net /CHANNEL_0: track 51.0 -> 18.2 mm
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Other:
- board text added: "Parameter X Parameter X Parameter X Parameter X Parameter X Parameter X Parameter X Parameter X Parameter X Parameter X"

Commit message: more routing...
Routing:
- net +3V3: track 0.00 -> 174.9 mm, vias 0 -> 4
- net /ADDRESS_SEND_B: track 59.4 -> 144.4 mm, vias 0 -> 1
- net /ADDRESS_SEND_A: track 67.8 -> 149.6 mm
- net /ADDRESS_SEND_C: track 50.8 -> 130.2 mm, vias 0 -> 1
- net /CONNECTION_SEND_A: track 0.00 -> 76.4 mm
- net /CONNECTION_READ_B: track 0.00 -> 70.9 mm, vias 0 -> 1
- net /CHANNEL_9: track 3.60 -> 71.7 mm, vias 0 -> 2
- net /CHANNEL_8: track 3.60 -> 69.9 mm, vias 0 -> 2
- net /CONNECTION_SEND_B: track 0.00 -> 57.6 mm
- net /CHANNEL_13: track 3.60 -> 59.6 mm, vias 0 -> 2
- net /CHANNEL_15: track 3.60 -> 56.4 mm, vias 0 -> 2
- net /CHANNEL_10: track 3.60 -> 55.9 mm, vias 0 -> 2
- net /CHANNEL_11: track 3.60 -> 55.6 mm, vias 0 -> 1
- net /CHANNEL_14: track 3.60 -> 53.7 mm, vias 0 -> 2
- net /CHANNEL_12: track 3.60 -> 51.2 mm, vias 0 -> 2
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
Commit message: think the hard routing is done...?
Routing:
- net /CHANNEL_3: track 17.0 -> 56.6 mm, vias 0 -> 2
- net /CHANNEL_0: track 18.2 -> 52.6 mm, vias 0 -> 2
- net /CHANNEL_1: track 23.5 -> 52.3 mm, vias 0 -> 2
- net /CHANNEL_7: track 27.2 -> 51.9 mm, vias 1 -> 3
- net /CHANNEL_2: track 26.6 -> 51.0 mm, vias 0 -> 2
- net /CHANNEL_4: track 37.7 -> 61.3 mm
- net /CHANNEL_5: track 24.5 -> 44.8 mm, vias 0 -> 2
- net /CHANNEL_6: track 27.2 -> 46.0 mm, vias 1 -> 2
- net /CHANNEL_9: track 71.7 -> 78.9 mm
- net /CHANNEL_8: track 69.9 -> 77.1 mm
- net /CHANNEL_12: track 51.2 -> 58.4 mm
- net /CHANNEL_11: track 55.6 -> 62.8 mm
- net /CHANNEL_10: track 55.9 -> 63.1 mm
- net /CHANNEL_15: track 56.4 -> 60.0 mm
- net /CHANNEL_14: track 53.7 -> 57.3 mm
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Other:
- board text added: "Parameter X Parameter X Parameter X Parameter X Parameter X Parameter X Parameter X Parameter X Parameter X Parameter X Parameter X Parameter X Parameter X Parameter X Parameter X Parameter X"
- board text removed: "Parameter X Parameter X Parameter X Parameter X Parameter X Parameter X Parameter X Parameter X Parameter X Parameter X"

Commit message: computer keeps crashing
Other:
- board size 200 x 100 mm -> 100 x 100 mm
Changed lines of the file:
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@@
       (net 50 "Net-(U2-Pad52)"))
   )
+  (gr_line (start 45 125) (end 45 25) (layer Edge.Cuts) (width 0.2))
+  (gr_line (start 145 125) (end 45 125) (layer Edge.Cuts) (width 0.2))
+  (gr_line (start 145 25) (end 145 125) (layer Edge.Cuts) (width 0.2))
+  (gr_line (start 45 25) (end 145 25) (layer Edge.Cuts) (width 0.2))
   (gr_text "Parameter X\nParameter X\nParameter X\nParameter X\nParameter X\nParameter X\nParameter X\nParameter X\nParameter X\nParameter X\nParameter X\nParameter X\nParameter X\nParameter X\nParameter X\nParameter X" (at 85.6 48) (layer F.SilkS)
     (effects (font (size 1.5 1.5) (thickness 0.3)))
   )
-  (gr_line (start 240 25) (end 40 25) (layer Edge.Cuts) (width 0.15))
-  (gr_line (start 240 125) (end 240 25) (layer Edge.Cuts) (width 0.15))
-  (gr_line (start 40 125) (end 240 125) (layer Edge.Cuts) (width 0.15))
-  (gr_line (start 40 25) (end 40 125) (layer Edge.Cuts) (width 0.15))
   (segment (start 91.415 72.555) (end 101.46 62.51) (width 0.25) (layer F.Cu) (net 5))
   (segment (start 56.7 72.555) (end 91.415 72.555) (width 0.25) (layer F.Cu) (net 5))

Commit message: moving things
Parts:
- moved D10 76.6 mm to (140.3, 70.5), turned to 180 degrees
- moved J5 74.9 mm to (139.0, 102.0), turned to 270 degrees
- moved D9 74.0 mm to (140.3, 66.4), turned to 180 degrees
- moved D8 71.9 mm to (140.3, 62.3), turned to 180 degrees
- moved R15 70.7 mm to (135.2, 70.5), turned to 180 degrees
- moved D7 70.3 mm to (140.3, 58.2), turned to 180 degrees
- moved D3 69.9 mm to (140.3, 41.9), turned to 180 degrees
- moved D6 69.3 mm to (140.3, 54.2), turned to 180 degrees
- moved D4 69.0 mm to (140.3, 45.9), turned to 180 degrees
- moved D5 68.8 mm to (140.3, 50.1), turned to 180 degrees
- moved R14 67.7 mm to (135.2, 66.4), turned to 180 degrees
- moved R13 65.3 mm to (135.2, 62.3), turned to 180 degrees
- moved R12 63.5 mm to (135.2, 58.2), turned to 180 degrees
- moved R8 62.7 mm to (135.2, 41.9), turned to 180 degrees
- moved R11 62.3 mm to (135.2, 54.2), turned to 180 degrees
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